File: PCB/td!40.kicad_pcb (KiCad board)
At the start: 2 copper layers, 0 parts

Commit message: PCB finished
Parts:
- added ?: , , F.Cu at (379.5, 226.2)
- added ?: , , F.Cu at (132.8, 187.7)
- added ?: , , F.Cu at (132.9, 226.9)
- added ?: , , F.Cu at (379.5, 187.5)
- added BT1: Battery_Cell, Connector_JST:JST_PH_S2B-PH-K_1x02_P2.00mm_Horizontal, B.Cu at (398.3, 213.6)
- added D1: D, Diode_SMD:D_SOD-123, B.Cu at (151.8, 174.7)
- added D10: D, Diode_SMD:D_SOD-123, B.Cu at (325.8, 174.7)
- added D11: D, Diode_SMD:D_SOD-123, B.Cu at (345.0, 174.7)
- added D12: D, Diode_SMD:D_SOD-123, B.Cu at (372.3, 174.7)
- added D13: D, Diode_SMD:D_SOD-123, B.Cu at (154.2, 194.1)
- added D14: D, Diode_SMD:D_SOD-123, B.Cu at (176.0, 194.0)
- added D15: D, Diode_SMD:D_SOD-123, B.Cu at (195.2, 194.0)
- added D16: D, Diode_SMD:D_SOD-123, B.Cu at (214.4, 194.0)
- added D17: D, Diode_SMD:D_SOD-123, B.Cu at (233.8, 194.0)
- added D18: D, Diode_SMD:D_SOD-123, B.Cu at (253.0, 194.0)
- added D19: D, Diode_SMD:D_SOD-123, B.Cu at (272.3, 194.1)
- added D2: D, Diode_SMD:D_SOD-123, B.Cu at (171.1, 174.7)
- added D20: D, Diode_SMD:D_SOD-123, B.Cu at (291.4, 194.1)
- added D21: D, Diode_SMD:D_SOD-123, B.Cu at (310.9, 194.1)
- added D22: D, Diode_SMD:D_SOD-123, B.Cu at (330.1, 194.1)
- added D23: D, Diode_SMD:D_SOD-123, B.Cu at (349.4, 194.1)
- added D24: D, Diode_SMD:D_SOD-123, B.Cu at (373.7, 194.1)
- added D25: D, Diode_SMD:D_SOD-123, B.Cu at (159.1, 213.5)
- added D26: D, Diode_SMD:D_SOD-123, B.Cu at (185.6, 213.5)
- added D27: D, Diode_SMD:D_SOD-123, B.Cu at (204.9, 213.5)
- added D28: D, Diode_SMD:D_SOD-123, B.Cu at (224.1, 213.5)
- added D29: D, Diode_SMD:D_SOD-123, B.Cu at (243.4, 213.5)
- added D3: D, Diode_SMD:D_SOD-123, B.Cu at (190.4, 174.7)
- added D30: D, Diode_SMD:D_SOD-123, B.Cu at (262.6, 213.4)
- added D31: D, Diode_SMD:D_SOD-123, B.Cu at (282.0, 213.7)
- added D32: D, Diode_SMD:D_SOD-123, B.Cu at (301.4, 213.7)
- added D33: D, Diode_SMD:D_SOD-123, B.Cu at (320.9, 213.7)
- added D34: D, Diode_SMD:D_SOD-123, B.Cu at (340.2, 213.7)
- added D35: D, Diode_SMD:D_SOD-123, B.Cu at (359.2, 213.7)
- added D36: D, Diode_SMD:D_SOD-123, B.Cu at (378.6, 213.7)
- added D37: D, Diode_SMD:D_SOD-123, B.Cu at (154.1, 232.9)
- added D38: D, Diode_SMD:D_SOD-123, B.Cu at (178.2, 232.9)
- added D39: D, Diode_SMD:D_SOD-123, B.Cu at (202.6, 232.9)
- added D4: D, Diode_SMD:D_SOD-123, B.Cu at (209.8, 174.8)
- added D40: D, Diode_SMD:D_SOD-123, B.Cu at (236.6, 232.9)
- added D41: D, Diode_SMD:D_SOD-123, B.Cu at (284.4, 232.9)
- added D43: D, Diode_SMD:D_SOD-123, B.Cu at (320.6, 233.1)
- added D44: D, Diode_SMD:D_SOD-123, B.Cu at (339.8, 233.1)
- added D45: D, Diode_SMD:D_SOD-123, B.Cu at (359.0, 233.1)
- added D46: D, Diode_SMD:D_SOD-123, B.Cu at (378.3, 233.1)
- added D47: D, Diode_SMD:D_SOD-123, B.Cu at (392.8, 230.9)
- added D5: D, Diode_SMD:D_SOD-123, B.Cu at (229.0, 174.8)
- added D6: D, Diode_SMD:D_SOD-123, B.Cu at (248.3, 174.8)
- added D7: D, Diode_SMD:D_SOD-123, B.Cu at (267.6, 174.7)
- added D8: D, Diode_SMD:D_SOD-123, B.Cu at (287.2, 174.7)
- added D9: D, Diode_SMD:D_SOD-123, B.Cu at (306.5, 174.7)
- added G***: LOGO, LOGO, F.Cu at (393.1, 212.7)
- added K1: KEYSW, crone:MX-Hotswap-1U, B.Cu at (143.2, 178.1)
- added K10: KEYSW, crone:MX-Hotswap-1U, B.Cu at (317.0, 178.1)
- added K11: KEYSW, crone:MX-Hotswap-1U, B.Cu at (336.3, 178.1)
- added K12: KEYSW, crone:MX-Hotswap-1.75U, B.Cu at (362.7, 178.1)
- added K13: KEYSW, crone:MX-Hotswap-1.25U, B.Cu at (145.6, 197.5)
- added K14: KEYSW, crone:MX-Hotswap-1U, B.Cu at (167.3, 197.5)
- added K15: KEYSW, crone:MX-Hotswap-1U, B.Cu at (186.6, 197.5)
- added K16: KEYSW, crone:MX-Hotswap-1U, B.Cu at (205.8, 197.5)
- added K17: KEYSW, crone:MX-Hotswap-1U, B.Cu at (225.0, 197.5)
- added K18: KEYSW, crone:MX-Hotswap-1U, B.Cu at (244.3, 197.5)
- added K19: KEYSW, crone:MX-Hotswap-1U, B.Cu at (263.6, 197.5)
- added K2: KEYSW, crone:MX-Hotswap-1U, B.Cu at (162.5, 178.1)
- added K20: KEYSW, crone:MX-Hotswap-1U, B.Cu at (282.9, 197.5)
- added K21: KEYSW, crone:MX-Hotswap-1U, B.Cu at (302.3, 197.5)
- added K22: KEYSW, crone:MX-Hotswap-1U, B.Cu at (321.6, 197.5)
- added K23: KEYSW, crone:MX-Hotswap-1U, B.Cu at (340.9, 197.5)
- added K24: KEYSW, crone:MX-Hotswap-1.5U, B.Cu at (365.1, 197.5)
- added K25: KEYSW, crone:MX-Hotswap-1.75U, B.Cu at (150.3, 217.0)
- added K26: KEYSW, crone:MX-Hotswap-1U, B.Cu at (176.7, 217.0)
- added K27: KEYSW, crone:MX-Hotswap-1U, B.Cu at (196.1, 217.0)
- added K28: KEYSW, crone:MX-Hotswap-1U, B.Cu at (215.3, 217.0)
- added K29: KEYSW, crone:MX-Hotswap-1U, B.Cu at (234.7, 217.0)
- added K3: KEYSW, crone:MX-Hotswap-1U, B.Cu at (181.8, 178.1)
- added K30: KEYSW, crone:MX-Hotswap-1U, B.Cu at (254.0, 217.0)
- added K31: KEYSW, crone:MX-Hotswap-1U, B.Cu at (273.3, 217.0)
- added K32: KEYSW, crone:MX-Hotswap-1U, B.Cu at (292.6, 217.0)
- added K33: KEYSW, crone:MX-Hotswap-1U, B.Cu at (312.0, 217.0)
- added K34: KEYSW, crone:MX-Hotswap-1U, B.Cu at (331.3, 217.0)
- added K35: KEYSW, crone:MX-Hotswap-1U, B.Cu at (350.6, 217.0)
- added K36: KEYSW, crone:MX-Hotswap-1U, B.Cu at (369.9, 217.0)
- added K37: KEYSW, crone:MX-Hotswap-1.25U, B.Cu at (145.5, 236.4)
- added K38: KEYSW, crone:MX-Hotswap-1.25U, B.Cu at (169.8, 236.4)
- added K39: KEYSW, crone:MX-Hotswap-1.25U, B.Cu at (194.1, 236.4)
- added K4: KEYSW, crone:MX-Hotswap-1U, B.Cu at (201.1, 178.1)
- added K40: KEYSW, crone:MX-Hotswap-2.25U-ReversedStabilizers, B.Cu at (227.9, 236.5)
- added K41: KEYSW, crone:MX-Hotswap-2.75U-ReversedStabilizers, B.Cu at (275.9, 236.5)
- added K42: KEYSW, crone:MX-Hotswap-1U, B.Cu at (311.9, 236.5)
- added K43: KEYSW, crone:MX-Hotswap-1U, B.Cu at (331.3, 236.4)
- added K44: KEYSW, crone:MX-Hotswap-1U, B.Cu at (350.5, 236.4)
- added K45: KEYSW, crone:MX-Hotswap-1U, B.Cu at (369.8, 236.4)
- added K5: KEYSW, crone:MX-Hotswap-1U, B.Cu at (220.4, 178.1)
- added K6: KEYSW, crone:MX-Hotswap-1U, B.Cu at (239.7, 178.1)
- added K7: KEYSW, crone:MX-Hotswap-1U, B.Cu at (259.1, 178.1)
- added K8: KEYSW, crone:MX-Hotswap-1U, B.Cu at (278.3, 178.1)
- added K9: KEYSW, crone:MX-Hotswap-1U, B.Cu at (297.7, 178.1)
- added L1: SK6812MINI, crone:YS-SK6812MINI-E, B.Cu at (362.8, 183.0)
- added L10: SK6812MINI, crone:YS-SK6812MINI-E, B.Cu at (181.9, 183.0)
- added L11: SK6812MINI, crone:YS-SK6812MINI-E, B.Cu at (162.5, 183.0)
- added L12: SK6812MINI, crone:YS-SK6812MINI-E, B.Cu at (143.2, 183.0)
- added L13: SK6812MINI, crone:YS-SK6812MINI-E, B.Cu at (145.5, 202.2)
- added L14: SK6812MINI, crone:YS-SK6812MINI-E, B.Cu at (167.3, 202.2)
- added L15: SK6812MINI, crone:YS-SK6812MINI-E, B.Cu at (186.5, 202.2)
- added L16: SK6812MINI, crone:YS-SK6812MINI-E, B.Cu at (205.8, 202.2)
- added L17: SK6812MINI, crone:YS-SK6812MINI-E, B.Cu at (225.0, 202.3)
- added L18: SK6812MINI, crone:YS-SK6812MINI-E, B.Cu at (244.3, 202.2)
- added L19: SK6812MINI, crone:YS-SK6812MINI-E, B.Cu at (263.5, 202.2)
- added L2: SK6812MINI, crone:YS-SK6812MINI-E, B.Cu at (336.3, 183.0)
- added L20: SK6812MINI, crone:YS-SK6812MINI-E, B.Cu at (283.0, 202.2)
- added L21: SK6812MINI, crone:YS-SK6812MINI-E, B.Cu at (302.2, 202.3)
- added L22: SK6812MINI, crone:YS-SK6812MINI-E, B.Cu at (321.5, 202.3)
- added L23: SK6812MINI, crone:YS-SK6812MINI-E, B.Cu at (340.8, 202.3)
- added L24: SK6812MINI, crone:YS-SK6812MINI-E, B.Cu at (365.0, 202.3)
- added L25: SK6812MINI, crone:YS-SK6812MINI-E, B.Cu at (369.8, 221.7)
- added L26: SK6812MINI, crone:YS-SK6812MINI-E, B.Cu at (350.5, 221.7)
- added L27: SK6812MINI, crone:YS-SK6812MINI-E, B.Cu at (331.3, 221.7)
- added L28: SK6812MINI, crone:YS-SK6812MINI-E, B.Cu at (312.0, 221.7)
- added L29: SK6812MINI, crone:YS-SK6812MINI-E, B.Cu at (292.5, 221.7)
- added L3: SK6812MINI, crone:YS-SK6812MINI-E, B.Cu at (317.0, 183.0)
- added L30: SK6812MINI, crone:YS-SK6812MINI-E, B.Cu at (273.3, 221.7)
- added L31: SK6812MINI, crone:YS-SK6812MINI-E, B.Cu at (254.0, 221.7)
- added L32: SK6812MINI, crone:YS-SK6812MINI-E, B.Cu at (234.8, 221.7)
- added L33: SK6812MINI, crone:YS-SK6812MINI-E, B.Cu at (215.3, 221.7)
- added L34: SK6812MINI, crone:YS-SK6812MINI-E, B.Cu at (196.1, 221.7)
- added L35: SK6812MINI, crone:YS-SK6812MINI-E, B.Cu at (176.8, 221.7)
- added L36: SK6812MINI, crone:YS-SK6812MINI-E, B.Cu at (150.3, 221.7)
- added L37: SK6812MINI, crone:YS-SK6812MINI-E, B.Cu at (145.5, 241.2)
- added L38: SK6812MINI, crone:YS-SK6812MINI-E, B.Cu at (169.8, 241.0)
- added L39: SK6812MINI, crone:YS-SK6812MINI-E, B.Cu at (194.0, 241.0)
- added L4: SK6812MINI, crone:YS-SK6812MINI-E, B.Cu at (297.5, 183.0)
- added L40: SK6812MINI, crone:YS-SK6812MINI-E, B.Cu at (228.0, 241.2)
- added L41: SK6812MINI, crone:YS-SK6812MINI-E, B.Cu at (275.8, 241.2)
- added L42: SK6812MINI, crone:YS-SK6812MINI-E, B.Cu at (311.8, 241.2)
- added L43: SK6812MINI, crone:YS-SK6812MINI-E, B.Cu at (331.3, 241.2)
- added L44: SK6812MINI, crone:YS-SK6812MINI-E, B.Cu at (350.5, 241.2)
- added L45: SK6812MINI, crone:YS-SK6812MINI-E, B.Cu at (369.8, 241.0)
- added L5: SK6812MINI, crone:YS-SK6812MINI-E, B.Cu at (278.3, 183.0)
- added L6: SK6812MINI, crone:YS-SK6812MINI-E, B.Cu at (259.0, 183.0)
- added L7: SK6812MINI, crone:YS-SK6812MINI-E, B.Cu at (239.8, 183.0)
- added L8: SK6812MINI, crone:YS-SK6812MINI-E, B.Cu at (220.3, 182.9)
- added L9: SK6812MINI, crone:YS-SK6812MINI-E, B.Cu at (201.0, 182.9)
- added OL1: OLED, crone:OLED, F.Cu at (393.2, 204.8)
- added R1: R, keebio:R_0805, B.Cu at (385.3, 202.8)
- added R2: R, keebio:R_0805, B.Cu at (385.3, 205.1)
- added RSW1: SW_PUSH, crone:ResetSW, B.Cu at (402.5, 212.7)
- added SW1: RotaryEncoder_Switch, keebio:RotaryEncoder_Alps_EC11E-Switch_Vertical_H20mm, F.Cu at (393.1, 228.2)
- added SW23: SW_DPDT, crone:switch-MSK-12C02-smd, F.Cu at (393.5, 167.9)
- added TOP_R: MountingHole_2.2mm_M2, MountingHole:MountingHole_2.2mm_M2, F.Cu at (382.0, 244.5)
- added TOP_R: MountingHole_2.2mm_M2, MountingHole:MountingHole_2.2mm_M2, F.Cu at (407.6, 244.5)
- added TOP_R: MountingHole_2.2mm_M2, MountingHole:MountingHole_2.2mm_M2, F.Cu at (407.5, 170.9)
- added TOP_R: MountingHole_2.2mm_M2, MountingHole:MountingHole_2.2mm_M2, F.Cu at (382.0, 170.9)
- added U1: nice_nano, Nice-nano:nice_nano, B.Cu at (393.3, 185.9)
Routing:
- net VCC: track 0.00 -> 1118.4 mm, vias 0 -> 5
- net col0: track 0.00 -> 406.8 mm, vias 0 -> 5
- net col1: track 0.00 -> 402.0 mm, vias 0 -> 10
- net col3: track 0.00 -> 380.8 mm, vias 0 -> 10
- net col2: track 0.00 -> 363.1 mm, vias 0 -> 11
- net col4: track 0.00 -> 340.9 mm, vias 0 -> 11
- net row3: track 0.00 -> 287.4 mm
- net col5: track 0.00 -> 274.9 mm, vias 0 -> 8
- net row2: track 0.00 -> 262.1 mm, vias 0 -> 1
- net row0: track 0.00 -> 257.6 mm, vias 0 -> 2
- net row1: track 0.00 -> 251.8 mm
- net row6: track 0.00 -> 149.2 mm, vias 0 -> 1
- net row5: track 0.00 -> 146.5 mm, vias 0 -> 2
- net row4: track 0.00 -> 133.1 mm, vias 0 -> 2
- net row7: track 0.00 -> 111.3 mm, vias 0 -> 1
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- added copper zone on B.Cu, net GND
- added copper zone on F.Cu, net GND
Other:
- board outline added: 282.1 x 81.3 mm

Commit message: Update: No more DRC errors, yayy
Parts:
- removed R1, R2: R, keebio:R_0805
- moved L25 0.15 mm to (369.9, 221.7)
- moved L4 0.14 mm to (297.7, 182.9)
- moved L32 0.13 mm to (234.7, 221.7)
- moved L44 0.13 mm to (350.5, 241.1)
- moved L20 0.12 mm to (282.9, 202.3)
- moved L43 0.12 mm to (331.2, 241.1)
- moved L37 0.12 mm to (145.5, 241.1)
- moved L1 0.12 mm to (362.7, 182.9)
- moved L3 0.11 mm to (317.0, 182.9)
- moved L19 0.11 mm to (263.6, 202.3)
- moved L42 0.11 mm to (311.9, 241.2)
- moved L7 0.11 mm to (239.7, 182.9)
- moved L10 0.11 mm to (181.8, 182.9)
- moved L5 0.10 mm to (278.4, 182.9)
- moved L45 0.09 mm to (369.9, 241.1)
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- renumbered TOP_R to M1, TOP_R to M2, TOP_R to M3, TOP_R to M4
Routing:
- net VCC: track 1118.4 -> 1074.9 mm
- net col3: track 380.8 -> 391.6 mm, vias 10 -> 9
- net SCL: track 31.0 -> 25.0 mm
- net col1: track 402.0 -> 407.3 mm
- net rot1: track 27.0 -> 31.0 mm
- net SDA: track 30.7 -> 27.9 mm
- net col5: track 274.9 -> 272.1 mm, vias 8 -> 6
- net Net-(L24-DIN): track 26.2 -> 23.6 mm
- net row7: track 111.3 -> 113.7 mm
- net row2: track 262.1 -> 260.6 mm
- net row1: track 251.8 -> 253.1 mm
- net row6: track 149.2 -> 150.5 mm
- net row0: track 257.6 -> 258.7 mm
- net row3: track 287.4 -> 288.5 mm

Commit message: Correct the RGB SK6812 pinout
Parts:
- BT1: footprint Connector_JST:JST_PH_S2B-PH-K_1x02_P2.00mm_Horizontal -> crone:JST_PH_S2B-PH-K_1x02_P2.00mm_Horizontal_flipped
- D1, D10, D11, D12, D13, D14, D15, D16, D17, D18, D19, D2, D20, D21, D22, D23, D24, D25, D26, D27, D28, D29, D3, D30, D31, D32, D33, D34, D35, D36, D37, D38, D39, D4, D40, D41, D5, D6, D7, D8, D9: value D -> ~
- D42: renamed from D43; value D -> ~
- D43: renamed from D44; value D -> ~
- D44: renamed from D45; value D -> ~
- D45: renamed from D46; value D -> ~
- SW23: value SW_DPDT -> SW23
- moved RSW1 0.50 mm to (403.0, 212.6)
- renumbered D47 to D46
Connections:
- net Battery renamed BAT
- net reset renamed RST
- L1 pad 1: unconnected-(L1-DOUT-Pad1) -> LED
- L45 pad 3: LED -> unconnected-(L45-DOUT-Pad3)
Routing:
- net LED: track 98.7 -> 40.1 mm, vias 2 -> 0
- net RST: track 55.9 -> 48.7 mm
- net Net-(BT1-+): track 61.6 -> 60.1 mm
- net row6: track 150.5 -> 151.3 mm
- net BAT: track 6.74 -> 7.31 mm
