File: PCB/td!40.kicad_sch (KiCad schematic)
At the start: 144 parts, among them K1 KEYSW, K10 KEYSW, K11 KEYSW, K12 KEYSW, K13 KEYSW, K14 KEYSW, K15 KEYSW, K16 KEYSW, K17 KEYSW, K18 KEYSW, K19 KEYSW, K2 KEYSW, K20 KEYSW, K21 KEYSW, K22 KEYSW, K23 KEYSW, K24 KEYSW, K25 KEYSW, K26 KEYSW, K27 KEYSW, K28 KEYSW, K29 KEYSW, K3 KEYSW, K30 KEYSW, K31 KEYSW, K32 KEYSW, K33 KEYSW, K34 KEYSW, K35 KEYSW, K36 KEYSW, K37 KEYSW, K38 KEYSW, K39 KEYSW, K4 KEYSW, K40 KEYSW, K41 KEYSW, K42 KEYSW, K43 KEYSW, K44 KEYSW, K45 KEYSW, K5 KEYSW, K6 KEYSW, K7 KEYSW, K8 KEYSW, K9 KEYSW, SW1 RotaryEncoder_Switch, SW2 SW_Push, SW3 SW_DPDT_x2, U1 nice_nano

Commit message: PCB finished
Parts:
- removed D1, D10, D11, D12, D13, D14, D15, D16, D17, D18, D19, D2, D20, D21, D22, D23, D24, D25, D26, D27, D28, D29, D3, D30, D31, D32, D33, D34, D35, D36, D37, D38, D39, D4, D40, D41, D42, D43, D44, D45, D46, D5, D6, D7, D8, D9: 1N4148WS, Diode_SMD:D_SOD-323, symbol Diode:1N4148WS
- removed SW2: SW_Push, crone:ResetSW, symbol Switch:SW_Push
- removed SW3: SW_DPDT_x2, crone:switch-MSK-12C02-smd, symbol Switch:SW_DPDT_x2
- removed U1: nice_nano, Nice-nano:nice_nano, symbol nice-nano:nice_nano
- added D1, D10, D11, D12, D13, D14, D15, D16, D17, D18, D19, D2, D20, D21, D22, D23, D24, D25, D26, D27, D28, D29, D3, D30, D31, D32, D33, D34, D35, D36, D37, D38, D39, D4, D40, D41, D42, D43, D44, D45, D5, D6, D7, D8, D9: (no value), Diode_SMD:D_SOD-123, symbol Device:D
- added D46: D, Diode_SMD:D_SOD-123, symbol Device:D
- added RSW1: SW_PUSH, crone:ResetSW, symbol crone:SW_PUSH
- added SW2: SW23, crone:switch-MSK-12C02-smd, symbol Switch:SW_DPDT_x2
- added U1: nice_nano, Nice-nano:nice_nano, symbol Nice-nano:nice_nano
Connections:
- net BAT: now also SW2.3 (C), U1.24 (BATIN/P0.04)
- net GND: now also RSW1.2, U1.23 (GND), U1.3 (GND), U1.4 (GND)
- net LED: now also U1.1 (TX0/P0.06)
- net RST: now also RSW1.1, U1.22 (RST)
- net SCL: now also U1.6 (P0.20)
- net SDA: now also U1.5 (P0.17)
- net VCC: now also U1.21 (VCC)
- net col0: now also U1.15 (P1.11)
- net col1: now also U1.10 (P0.11)
- net col2: now also U1.16 (P1.13)
- net col3: now also U1.9 (P1.00)
- net col4: now also U1.17 (P1.15)
- net col5: now also U1.8 (P0.24)
- net rot0: now also U1.31 (P1.01)
- net rot1: now also U1.33 (P1.07)
- net row0: now also D1.1 (K), D2.1 (K), D3.1 (K), D4.1 (K), D5.1 (K), D6.1 (K), U1.19 (AIN5/P0.29)
- net row1: now also D13.1 (K), D14.1 (K), D15.1 (K), D16.1 (K), D17.1 (K), D18.1 (K), U1.18 (AIN0/P0.02)
- net row2: now also D25.1 (K), D26.1 (K), D27.1 (K), D28.1 (K), D29.1 (K), D30.1 (K), U1.14 (NFC2/P0.10)
- net row3: now also D37.1 (K), D38.1 (K), D39.1 (K), D40.1 (K), D41.1 (K), U1.12 (P1.06)
- net row4: now also D10.1 (K), D11.1 (K), D12.1 (K), D7.1 (K), D8.1 (K), D9.1 (K), U1.20 (AIN7/P0.31)
- net row5: now also D19.1 (K), D20.1 (K), D21.1 (K), D22.1 (K), D23.1 (K), D24.1 (K), U1.7 (P0.22)
- net row6: now also D31.1 (K), D32.1 (K), D33.1 (K), D34.1 (K), D35.1 (K), D36.1 (K), U1.11 (P1.04)
- net row7: now also D42.1 (K), D43.1 (K), D44.1 (K), D45.1 (K), D46.1 (K), U1.13 (NFC1/P0.09)
- net at K24.2: now also D24.2 (A)
- net at K30.2: now also D30.2 (A)
- net at K41.2: now also D41.2 (A)
- net at K37.2: now also D37.2 (A)
- net at K12.2: now also D12.2 (A)
- net at K38.2: now also D38.2 (A)
- net at K25.2: now also D25.2 (A)
- net at K28.2: now also D28.2 (A)
- net at K43.2: now also D43.2 (A)
- net at K13.2: now also D13.2 (A)
- net at BT1.1 (+): now also SW2.2 (B)
- net at K10.2: now also D10.2 (A)
- net at K5.2: now also D5.2 (A)
- net at K23.2: now also D23.2 (A)
- net at K33.2: now also D33.2 (A)
- net at K6.2: now also D6.2 (A)
- net at K15.2: now also D15.2 (A)
- net at K2.2: now also D2.2 (A)
- net at K42.2: now also D42.2 (A)
- net at K29.2: now also D29.2 (A)
- net at K4.2: now also D4.2 (A)
- net at K18.2: now also D18.2 (A)
- net at K21.2: now also D21.2 (A)
- net at K8.2: now also D8.2 (A)
- net at K3.2: now also D3.2 (A)
- net at K44.2: now also D44.2 (A)
- net at K45.2: now also D45.2 (A)
- net at K35.2: now also D35.2 (A)
- net at K26.2: now also D26.2 (A)
- net at K27.2: now also D27.2 (A)
- net at SW1.S2: now also D46.2 (A)
- net at K20.2: now also D20.2 (A)
- net at K32.2: now also D32.2 (A)
- net at K11.2: now also D11.2 (A)
- net at K36.2: now also D36.2 (A)
- net at K34.2: now also D34.2 (A)
- net at K22.2: now also D22.2 (A)
- net at K16.2: now also D16.2 (A)
- net at K17.2: now also D17.2 (A)
- net at K1.2: now also D1.2 (A)
- net at K31.2: now also D31.2 (A)
- net at K40.2: now also D40.2 (A)
- net at K9.2: now also D9.2 (A)
- net at K19.2: now also D19.2 (A)
- net at K7.2: now also D7.2 (A)
- net at K39.2: now also D39.2 (A)
- net at K14.2: now also D14.2 (A)
Other:
- moved on the sheet: BT1, OL1, R1, R2, SW1

Commit message: Correct the RGB SK6812 pinout
Parts:
- removed R1, R2: R, keebio:R_0805, symbol Device:R
- BT1: footprint Connector_JST:JST_PH_S2B-PH-K_1x02_P2.00mm_Horizontal -> crone:JST_PH_S2B-PH-K_1x02_P2.00mm_Horizontal_flipped
- D1, D10, D11, D12, D13, D14, D15, D16, D17, D18, D19, D2, D20, D21, D22, D23, D24, D25, D26, D27, D28, D29, D3, D30, D31, D32, D33, D34, D35, D36, D37, D38, D39, D4, D40, D41, D42, D43, D44, D45, D5, D6, D7, D8, D9: value (none) -> ~
- renumbered SW2 to SW23
Connections:
- net LED: now also L1.1 (DIN); no longer L45.3 (DIN)
